Commit message: v0.0.1 完成 A2 与 VX300S 合并

File: a2-arm.urdf.xacro (robot description, xacro)
@@ -6,6 +6,6 @@
     before the xacro:a2 / xacro:vx300s calls below can work.
   -->
-  <xacro:include filename="$(find combine)/a2.urdf.xacro"/>
-  <xacro:include filename="$(find combine)/vx300s.urdf.xacro"/>
+  <xacro:include filename="a2.urdf.xacro"/>
+  <xacro:include filename="vx300s.urdf.xacro"/>
   <!--
     Expected link names in the current models:

File: a2.urdf.xacro (robot description, xacro)
@@ -1,3 +1,5 @@
-<robot name="a2">
+<?xml version="1.0"?>
+<robot name="a2" xmlns:xacro="http://www.ros.org/wiki/xacro">
+  <xacro:macro name="a2">
   <!-- [CAUTION] uncomment when convert to mujoco -->
   <!-- <mujoco>
@@ -1022,3 +1024,4 @@
       xyz="0 0 0" />
   </joint>
+  </xacro:macro>
 </robot>

File: vx300s.urdf.xacro (robot description, xacro)
@@ -1,4 +1,5 @@
 <?xml version="1.0" ?>
-<robot name="vx300s">
+<robot name="vx300s" xmlns:xacro="http://www.ros.org/wiki/xacro">
+  <xacro:macro name="vx300s">
   <material name="interbotix_black">
     <texture filename="meshes/interbotix_black.png"/>
@@ -420,3 +421,4 @@
     </inertial>
   </link>
+  </xacro:macro>
 </robot>
