Commit message: v0.0.3 锁死旋转 gripper

File: a2-vx300s.urdf (robot description, URDF)
Before this commit: robot a2_vx300s, 31 links, 30 joints
Joints:
- joint gripper: type continuous -> fixed

Commit message: add mujoco compiler to visualize in mujoco

File: a2-vx300s.urdf (robot description, URDF)
Before this commit: robot a2_vx300s, 31 links, 30 joints
Links:
- added link world
Joints:
- added joint floating_base_joint: type floating, parent world, child base_link

File: a2.urdf (robot description, URDF)
Before this commit: robot a2, 17 links, 16 joints
Links:
- added link world
Joints:
- added joint floating_base_joint: type floating, parent world, child base_link

File: vx300s.urdf (robot description, URDF)
Before this commit: robot vx300s, 14 links, 13 joints
Links:
- added link world
Joints:
- added joint floating_base_joint: type floating, parent world, child vx300s/base_link
