Commit message: add: a2-arm-wbc

File: urdf/a2-vx300s-wbc.urdf (robot description, URDF)
Before this commit: robot a2_vx300s, 31 links, 30 joints
Joints:
- joint left_finger: origin xyz=0 0.0085 0 rpy=0 0 0 -> xyz=0 0.0445 0 rpy=0 0 0; type prismatic -> fixed
- joint right_finger: origin xyz=0 -0.0085 0 rpy=0 0 0 -> xyz=0 -0.0445 0 rpy=0 0 0; type prismatic -> fixed
