Commit message: 修改 A2-ARM (后移 Arm base 8cm)

File: urdf/a2-vx300s.urdf (robot description, URDF)
Before this commit: robot a2_vx300s, 31 links, 30 joints
Joints:
- joint arm_mount_joint: origin xyz=0.20 0 0.16 rpy=0 0 0 -> xyz=0.08 0 0.16 rpy=0 0 0

Commit message: fixbug: A2-ARM 修改 finger link 初始位置

File: urdf/a2-vx300s.urdf (robot description, URDF)
Before this commit: robot a2_vx300s, 31 links, 30 joints
Joints:
- joint left_finger: limit lower=0.021 upper=0.057 effort=5 velocity=1 -> lower=0 upper=0.036 effort=5 velocity=1; origin xyz=0 0 0 rpy=0 0 0 -> xyz=0 0.021 0 rpy=0 0 0
- joint right_finger: limit lower=-0.057 upper=-0.021 effort=5 velocity=1 -> lower=-0.036 upper=0 effort=5 velocity=1; origin xyz=0 0 0 rpy=0 0 0 -> xyz=0 -0.021 0 rpy=0 0 0

File: urdf/vx300s.urdf.xacro (robot description, xacro)
@@ -336,6 +336,6 @@
   <joint name="left_finger" type="prismatic">
     <axis xyz="0 1 0"/>
-    <limit effort="5" lower="0.021" upper="0.057" velocity="1"/>
-    <origin rpy="0 0 0" xyz="0 0 0"/>
+    <limit effort="5" lower="0" upper="0.036" velocity="1"/>
+    <origin rpy="0 0 0" xyz="0 0.021 0"/>
     <parent link="vx300s/fingers_link"/>
     <child link="vx300s/left_finger_link"/>
@@ -373,6 +373,6 @@
   <joint name="right_finger" type="prismatic">
     <axis xyz="0 1 0"/>
-    <limit effort="5" lower="-0.057" upper="-0.021" velocity="1"/>
-    <origin rpy="0 0 0" xyz="0 0 0"/>
+    <limit effort="5" lower="-0.036" upper="0" velocity="1"/>
+    <origin rpy="0 0 0" xyz="0 -0.021 0"/>
     <parent link="vx300s/fingers_link"/>
     <child link="vx300s/right_finger_link"/>

Commit message: fixbug: A2-ARM 修改 finger link 原点位置

File: urdf/a2-vx300s.urdf (robot description, URDF)
Before this commit: robot a2_vx300s, 31 links, 30 joints
Joints:
- joint left_finger: limit lower=0 upper=0.036 effort=5 velocity=1 -> lower=0.0 upper=0.036 effort=5 velocity=1; origin xyz=0 0.021 0 rpy=0 0 0 -> xyz=0 0.0085 0 rpy=0 0 0
- joint right_finger: limit lower=-0.036 upper=0 effort=5 velocity=1 -> lower=-0.036 upper=-0.0 effort=5 velocity=1; origin xyz=0 -0.021 0 rpy=0 0 0 -> xyz=0 -0.0085 0 rpy=0 0 0

File: urdf/vx300s.urdf.xacro (robot description, xacro)
@@ -336,6 +336,6 @@
   <joint name="left_finger" type="prismatic">
     <axis xyz="0 1 0"/>
-    <limit effort="5" lower="0" upper="0.036" velocity="1"/>
-    <origin rpy="0 0 0" xyz="0 0.021 0"/>
+    <limit effort="5" lower="0.0" upper="0.036" velocity="1"/>
+    <origin rpy="0 0 0" xyz="0 0.0085 0"/>
     <parent link="vx300s/fingers_link"/>
     <child link="vx300s/left_finger_link"/>
@@ -353,5 +353,5 @@
   <link name="vx300s/left_finger_link">
     <visual>
-      <origin rpy="1.5707963267948966 -3.141592653589793 1.5707963267948966" xyz="-0.0404 -0.0575 0"/>
+      <origin rpy="1.5707963267948966 -3.141592653589793 1.5707963267948966" xyz="-0.0404 -0.045 0"/>
       <geometry>
         <mesh filename="meshes/vx300s_10_gripper_finger.stl" scale="0.001 0.001 0.001"/>
@@ -360,5 +360,5 @@
     </visual>
     <collision>
-      <origin rpy="1.5707963267948966 -3.141592653589793 1.5707963267948966" xyz="-0.0404 -0.0575 0"/>
+      <origin rpy="1.5707963267948966 -3.141592653589793 1.5707963267948966" xyz="-0.0404 -0.045 0"/>
       <geometry>
         <mesh filename="meshes/vx300s_10_gripper_finger.stl" scale="0.001 0.001 0.001"/>
@@ -366,5 +366,5 @@
     </collision>
     <inertial>
-      <origin rpy="3.141592653589793 3.141592653589793 1.5707963267948966" xyz="0.0173440000 -0.0060692000 0.0000000000"/>
+      <origin rpy="3.141592653589793 3.141592653589793 1.5707963267948966" xyz="0.0173440000 0.0064308000 0.0000000000"/>
       <mass value="0.034796"/>
       <inertia ixx="0.0000243300" iyy="0.0000125500" izz="0.0000141700" ixy="-0.0000024004" ixz="0.0000000000" iyz="0.0000000000"/>
@@ -373,6 +373,6 @@
   <joint name="right_finger" type="prismatic">
     <axis xyz="0 1 0"/>
-    <limit effort="5" lower="-0.036" upper="0" velocity="1"/>
-    <origin rpy="0 0 0" xyz="0 -0.021 0"/>
+    <limit effort="5" lower="-0.036" upper="-0.0" velocity="1"/>
+    <origin rpy="0 0 0" xyz="0 -0.0085 0"/>
     <parent link="vx300s/fingers_link"/>
     <child link="vx300s/right_finger_link"/>
@@ -391,5 +391,5 @@
   <link name="vx300s/right_finger_link">
     <visual>
-      <origin rpy="-1.5707963267948966 3.141592653589793 -1.5707963267948966" xyz="-0.0404 0.0575 0 "/>
+      <origin rpy="-1.5707963267948966 3.141592653589793 -1.5707963267948966" xyz="-0.0404 0.045 0"/>
       <geometry>
         <mesh filename="meshes/vx300s_10_gripper_finger.stl" scale="0.001 0.001 0.001"/>
@@ -398,5 +398,5 @@
     </visual>
     <collision>
-      <origin rpy="-1.5707963267948966 3.141592653589793 -1.5707963267948966" xyz="-0.0404 0.0575 0 "/>
+      <origin rpy="-1.5707963267948966 3.141592653589793 -1.5707963267948966" xyz="-0.0404 0.045 0"/>
       <geometry>
         <mesh filename="meshes/vx300s_10_gripper_finger.stl" scale="0.001 0.001 0.001"/>
@@ -404,5 +404,5 @@
     </collision>
     <inertial>
-      <origin rpy="0 3.141592653589793 1.5707963267948966" xyz="0.0173440000 0.0060692000  0.0000000000"/>
+      <origin rpy="0 3.141592653589793 1.5707963267948966" xyz="0.0173440000 -0.0064308000 0.0000000000"/>
       <mass value="0.034796"/>
       <inertia ixx="0.0000243300" iyy="0.0000125500" izz="0.0000141700" ixy="0.0000024001" ixz="0.0000000000" iyz="0.0000000000"/>

Commit message: perf: A2-ARM 碰撞体积

File: urdf/a2-vx300s.urdf (robot description, URDF)
Before this commit: robot a2_vx300s, 31 links, 30 joints
Links:
- link vx300s/base_link: geometry collision box size=0.115 0.082 0.045; collision cylinder length=0.067 radius=0.069
- link vx300s/gripper_bar_link: geometry visual mesh filename=meshes/vx300s_9_gripper_bar.stl scale=0.001 0.001 0.001
- link vx300s/gripper_link: geometry collision box size=0.0447 0.150 0.046; visual mesh filename=meshes/vx300s_7_gripper.stl scale=0.001 0.001 0.001
- link vx300s/gripper_prop_link: geometry visual mesh filename=meshes/vx300s_8_gripper_prop.stl scale=0.001 0.001 0.001
- link vx300s/left_finger_link: geometry collision box size=0.06 0.0205 0.061; visual mesh filename=meshes/vx300s_10_gripper_finger.stl scale=0.001 0.001 0.001
- link vx300s/lower_forearm_link: geometry collision box size=0.118 0.1 0.0395; visual mesh filename=meshes/vx300s_5_lower_forearm.stl scale=0.001 0.001 0.001
- link vx300s/right_finger_link: geometry collision box size=0.06 0.0205 0.061; visual mesh filename=meshes/vx300s_10_gripper_finger.stl scale=0.001 0.001 0.001
- link vx300s/shoulder_link: geometry collision box size=0.0335 0.102 0.0585; visual mesh filename=meshes/vx300s_2_shoulder.stl scale=0.001 0.001 0.001
- link vx300s/upper_arm_link: geometry collision box size=0.020 0.040 0.295; collision box size=0.06375 0.1012 0.0419
- link vx300s/upper_forearm_link: geometry collision box size=0.166791 0.0452 0.0315; visual mesh filename=meshes/vx300s_4_upper_forearm.stl scale=0.001 0.001 0.001
- link vx300s/wrist_link: geometry collision box size=0.034 0.055 0.0465; visual mesh filename=meshes/vx300s_6_wrist.stl scale=0.001 0.001 0.001
